File: samd51_breakout.sch (KiCad schematic (older format))
At the start: 22 parts, among them J1 Conn_SWD, J2 USB_C_Receptacle_USB2.0, J3 Conn_01x19, J4 Conn_02x07_Counter_Clockwise, J5 Conn_01x19, U1 ATSAMD51J, U2 XC6206P332MR

Commit message: Rename schematic, add more photos
Parts:
- J2: symbol Connector:USB_C_Receptacle_USB2.0 -> samd51_breakout-rescue:USB_C_Receptacle_USB2.0-Connector
Changed lines of the file:
@@
 EESchema Schematic File Version 4
+LIBS:samd51_breakout-cache
 EELAYER 29 0
 EELAYER END
@@
 	7650 2250 7500 2250
 $Comp
-L Connector:USB_C_Receptacle_USB2.0 J2
+L samd51_breakout-rescue:USB_C_Receptacle_USB2.0-Connector J2
 U 1 1 5C182564
 P 1650 2000
